Commit message: update

File: src/covid_robot_description/urdf/covid_robot_backup.urdf.xacro (robot description, xacro)
@@ -55,5 +55,5 @@
     <parent link="base_link"/>
     <child link="wheel_left_link_4"/>
-    <origin xyz="-0.45 0.22 0.023" rpy="0 1.57 0"/>
+    <origin xyz="-0.40 0.33 0.023" rpy="-1.57 0 0"/>
     <axis xyz="0 0 1"/>
   </joint>
@@ -100,5 +100,5 @@
     <parent link="base_link"/>
     <child link="wheel_left_link"/>
-    <origin xyz="0.45 0.22 0.023" rpy="0 -1.57 0"/>
+    <origin xyz="0.40 0.33 0.023" rpy="-1.57 0 0"/>
     <axis xyz="0 0 1"/>
   </joint>
@@ -145,5 +145,5 @@
     <parent link="base_link"/>
     <child link="wheel_right_link"/>
-    <origin xyz="0.45 -0.22 0.023" rpy="0 -1.57 0"/>
+    <origin xyz="0.40 -0.27 0.023" rpy="-1.57 0 0"/>
     <axis xyz="0 0 1"/>
   </joint>
@@ -190,5 +190,5 @@
     <parent link="base_link"/>
     <child link="wheel_right_link_1"/>
-    <origin xyz="-0.45 -0.22 0.023" rpy="0 1.57 0"/>
+    <origin xyz="-0.40 -0.27 0.023" rpy="-1.57 0 0"/>
     <axis xyz="0 0 1"/>
   </joint>
@@ -199,69 +199,19 @@
         <mesh filename="package://covid_robot_description/meshes/wheels/covid_robot_tire.stl" scale="0.001 0.001 0.001"/>
       </geometry>
-    </visual>
-    <collision>
-      <origin xyz="0 0 0" rpy="0 0 0"/>
-      <geometry>
-        <cylinder length="0.018" radius="0.033"/>
-      </geometry>
-    </collision>
-    <inertial>
-      <origin xyz="0 0 0" />
-      <mass value="2.8498940e-02" />
-      <inertia ixx="1.1175580e-05" ixy="-4.2369783e-11" ixz="-5.9381719e-09"
-               iyy="1.1192413e-05" iyz="-1.4400107e-11"
-               izz="2.0712558e-05" />
-      </inertial>
-  </link>
-  <joint name="body_side_left" type="fixed">
-    <parent link="base_link"/>
-    <child link="body_side_left"/>
-    <origin xyz="-0.30 0.0 0.460" rpy="0 0 0"/>
-  </joint>
-  <link name="body_side_left">
-    <visual>
-      <origin xyz="-0.3 0.1 0.1" rpy="1.57 0 0"/>
-      <geometry>
-        <mesh filename="package://covid_robot_description/meshes/bases/body_side.stl" scale="0.001 0.001 0.001"/>
-      </geometry>
-      <material name="dark"/>
-    </visual>
-    <collision>
-      <origin xyz="0 0 0" rpy="0 0 0"/>
-    </collision>
-  </link>
-  <joint name="body_side_right" type="fixed">
-    <parent link="base_link"/>
-    <child link="body_side_right"/>
-    <origin xyz="0.30 0.0 0.460" rpy="0 0 0"/>
-  </joint>
-  <link name="body_side_right">
-    <visual>
-      <origin xyz="0.1 0.1 0.1" rpy="1.57 0 0"/>
-      <geometry>
-        <mesh filename="package://covid_robot_description/meshes/bases/body_side.stl" scale="0.001 0.001 0.001"/>
-      </geometry>
-      <material name="dark"/>
-    </visual>
-    <collision>
-      <origin xyz="0 0 0" rpy="0 0 0"/>
-    </collision>
-  </link>
-  <joint name="body_side_rack_left" type="fixed">
-    <parent link="base_link"/>
-    <child link="body_side_rack_left"/>
-    <origin xyz="-0.30 0.0 0.835" rpy="0 1.57 1.57"/>
-  </joint>
-  <link name="body_side_rack_left">
-    <visual>
-      <origin xyz="0 0 0.1" rpy="1.57 0 0"/>
-      <geometry>
-        <mesh filename="package://covid_robot_description/meshes/bases/body_side_rack.stl" scale="0.001 0.001 0.001"/>
-      </geometry>
-      <material name="dark"/>
-    </visual>
-    <collision>
-      <origin xyz="0 0 0" rpy="0 0 0"/>
-    </collision>
+      <material name="dark"/>
+    </visual>
+    <collision>
+      <origin xyz="0 0 0" rpy="0 0 0"/>
+      <geometry>
+        <cylinder length="0.018" radius="0.033"/>
+      </geometry>
+    </collision>
+    <inertial>
+      <origin xyz="0 0 0" />
+      <mass value="2.8498940e-02" />
+      <inertia ixx="1.1175580e-05" ixy="-4.2369783e-11" ixz="-5.9381719e-09"
+               iyy="1.1192413e-05" iyz="-1.4400107e-11"
+               izz="2.0712558e-05" />
+      </inertial>
   </link>
   <joint name="caster_back_right_joint" type="fixed">
