Commit message: backup

File: src/covid_robot_description/urdf/covid_robot.gazebo_backup.xacro (robot description, xacro)
@@ -1,7 +1,6 @@
 <?xml version="1.0"?>
 <robot name="covid_robot" xmlns:xacro="http://ros.org/wiki/xacro">
-  <xacro:arg name="laser_visual"  default="false"/>
-  <xacro:arg name="camera_visual" default="false"/>
-  <xacro:arg name="imu_visual"    default="false"/>
+  <xacro:arg name="laser_visual" default="false"/>
+  <xacro:arg name="imu_visual"   default="false"/>
   <gazebo reference="base_link">
     <material>Gazebo/DarkGrey</material>
@@ -27,32 +26,5 @@
     <material>Gazebo/FlatBlack</material>
   </gazebo>
-  <gazebo reference="wheel_left_link_4">
-    <material>Gazebo/FlatBlack</material>
-  </gazebo>
-  <gazebo reference="wheel_right_link_1">
-    <material>Gazebo/FlatBlack</material>
-  </gazebo>
-  <gazebo reference="wheel_left_link_4_steer">
-    <material>Gazebo/FlatBlack</material>
-  </gazebo>
-  <gazebo reference="wheel_right_link_1_steer">
-    <material>Gazebo/FlatBlack</material>
-  </gazebo>
-  <gazebo reference="wheel_left_link_steer">
-    <material>Gazebo/FlatBlack</material>
-  </gazebo>
-  <gazebo reference="wheel_right_link_steer">
-    <material>Gazebo/FlatBlack</material>
-  </gazebo>
-  <gazebo reference="caster_back_right_link">
-    <mu1>0.1</mu1>
-    <mu2>0.1</mu2>
-    <kp>1000000.0</kp>
-    <kd>100.0</kd>
-    <minDepth>0.001</minDepth>
-    <maxVel>1.0</maxVel>
-    <material>Gazebo/FlatBlack</material>
-  </gazebo>
-  <gazebo reference="caster_back_left_link">
+  <gazebo reference="caster_back_link">
     <mu1>0.1</mu1>
     <mu2>0.1</mu2>
@@ -68,8 +40,8 @@
       <visualize>$(arg imu_visual)</visualize>
     </sensor>
-    <material>Gazebo/Grey</material>
+    <material>Gazebo/FlatBlack</material>
   </gazebo>
   <gazebo>
-    <plugin name="turtlebot3_waffle_controller" filename="libgazebo_ros_diff_drive.so">
+    <plugin name="turtlebot3_burger_controller" filename="libgazebo_ros_diff_drive.so">
       <commandTopic>cmd_vel</commandTopic>
       <odometryTopic>odom</odometryTopic>
@@ -85,5 +57,5 @@
       <leftJoint>wheel_left_joint</leftJoint>
       <rightJoint>wheel_right_joint</rightJoint>
-      <wheelSeparation>0.287</wheelSeparation>
+      <wheelSeparation>0.160</wheelSeparation>
       <wheelDiameter>0.066</wheelDiameter>
       <wheelAcceleration>1</wheelAcceleration>
@@ -152,46 +124,3 @@
     </sensor>
   </gazebo>
-  <gazebo reference="camera_rgb_frame">
-    <sensor type="depth" name="realsense_R200">
-      <always_on>true</always_on>
-      <visualize>$(arg camera_visual)</visualize>
-      <camera>
-          <horizontal_fov>1.3439</horizontal_fov>
-          <image>
-              <width>1920</width>
-              <height>1080</height>
-              <format>R8G8B8</format>
-          </image>
-          <depth_camera></depth_camera>
-          <clip>
-              <near>0.03</near>
-              <far>100</far>
-          </clip>
-      </camera>
-      <plugin name="camera_controller" filename="libgazebo_ros_openni_kinect.so">
-        <baseline>0.2</baseline>
-        <alwaysOn>true</alwaysOn>
-        <updateRate>30.0</updateRate>
-        <cameraName>camera</cameraName>
-        <frameName>camera_rgb_optical_frame</frameName>
-        <imageTopicName>rgb/image_raw</imageTopicName>
-        <depthImageTopicName>depth/image_raw</depthImageTopicName>
-        <pointCloudTopicName>depth/points</pointCloudTopicName>
-        <cameraInfoTopicName>rgb/camera_info</cameraInfoTopicName>
-        <depthImageCameraInfoTopicName>depth/camera_info</depthImageCameraInfoTopicName>
-        <pointCloudCutoff>0.4</pointCloudCutoff>
-            <hackBaseline>0.07</hackBaseline>
-            <distortionK1>0.0</distortionK1>
-            <distortionK2>0.0</distortionK2>
-            <distortionK3>0.0</distortionK3>
-            <distortionT1>0.0</distortionT1>
-            <distortionT2>0.0</distortionT2>
-        <CxPrime>0.0</CxPrime>
-        <Cx>0.0</Cx>
-        <Cy>0.0</Cy>
-        <focalLength>0</focalLength>
-        <hackBaseline>0</hackBaseline>
-      </plugin>
-    </sensor>
-  </gazebo>
 </robot>

File: src/covid_robot_description/urdf/covid_robot_backup2.urdf.xacro (robot description, xacro)
@@ -23,5 +23,5 @@
       <origin xyz="0.0 0 0.047" rpy="0 0 0"/>
       <geometry>
-        <box size="1.0 1.0 0.093"/>
+        <box size="1.0 1.0 0.094"/>
       </geometry>
     </collision>
@@ -59,5 +59,5 @@
   <link name="wheel_left_link_4">
     <visual>
-      <origin xyz="0 0 0.02" rpy="1.57 0 0"/>
+      <origin xyz="0 0 0" rpy="1.57 0 0"/>
       <geometry>
         <mesh filename="package://covid_robot_description/meshes/wheels/covid_robot_tire.stl" scale="0.001 0.001 0.001"/>
@@ -104,5 +104,5 @@
   <link name="wheel_left_link">
     <visual>
-      <origin xyz="0 0 0.02" rpy="1.57 0 0"/>
+      <origin xyz="0 0 0" rpy="1.57 0 0"/>
       <geometry>
         <mesh filename="package://covid_robot_description/meshes/wheels/covid_robot_tire.stl" scale="0.001 0.001 0.001"/>
@@ -149,5 +149,5 @@
   <link name="wheel_right_link">
     <visual>
-      <origin xyz="0 0 0.02" rpy="1.57 0 0"/>
+      <origin xyz="0 0 0" rpy="1.57 0 0"/>
       <geometry>
         <mesh filename="package://covid_robot_description/meshes/wheels/covid_robot_tire.stl" scale="0.001 0.001 0.001"/>
@@ -194,5 +194,5 @@
   <link name="wheel_right_link_1">
     <visual>
-      <origin xyz="0 0 0.02" rpy="1.57 0 0"/>
+      <origin xyz="0 0 0" rpy="1.57 0 0"/>
       <geometry>
         <mesh filename="package://covid_robot_description/meshes/wheels/covid_robot_tire.stl" scale="0.001 0.001 0.001"/>
@@ -312,5 +312,5 @@
     <parent link="base_link"/>
     <child link="base_scan"/>
-    <origin xyz="-0.064 0 0.2" rpy="0 0 0"/>
+    <origin xyz="-0.064 0 0.122" rpy="0 0 0"/>
   </joint>
   <link name="base_scan">
