Commit message: backup

File: src/covid_robot_description/urdf/covid_robot.gazebo.xacro (robot description, xacro)
@@ -5,5 +5,5 @@
   <xacro:arg name="imu_visual"    default="false"/>
   <gazebo reference="base_link">
-    <material>Gazebo/DarkGrey</material>
+    <material>Gazebo/FlatBlack</material>
   </gazebo>
   <gazebo reference="wheel_left_link">
@@ -15,5 +15,5 @@
     <maxVel>0.1</maxVel>
     <fdir1>1 0 0</fdir1>
-    <material>Gazebo/FlatBlack</material>
+    <material>Gazebo/DarkGrey</material>
   </gazebo>
   <gazebo reference="wheel_right_link">
@@ -25,23 +25,31 @@
     <maxVel>0.1</maxVel>
     <fdir1>1 0 0</fdir1>
-    <material>Gazebo/FlatBlack</material>
-  </gazebo>
-  <gazebo reference="wheel_left_link_4">
-    <material>Gazebo/FlatBlack</material>
+    <material>Gazebo/DarkGrey</material>
+  </gazebo>
+  <gazebo reference="wheel_left_link_1">
+    <material>Gazebo/DarkGrey</material>
   </gazebo>
   <gazebo reference="wheel_right_link_1">
-    <material>Gazebo/FlatBlack</material>
-  </gazebo>
-  <gazebo reference="wheel_left_link_4_steer">
-    <material>Gazebo/FlatBlack</material>
+    <material>Gazebo/DarkGrey</material>
+  </gazebo>
+  <gazebo reference="wheel_left_link_1_steer">
+    <material>Gazebo/DarkGrey</material>
   </gazebo>
   <gazebo reference="wheel_right_link_1_steer">
-    <material>Gazebo/FlatBlack</material>
+    <material>Gazebo/DarkGrey</material>
   </gazebo>
   <gazebo reference="wheel_left_link_steer">
-    <material>Gazebo/FlatBlack</material>
+    <material>Gazebo/DarkGrey</material>
   </gazebo>
   <gazebo reference="wheel_right_link_steer">
-    <material>Gazebo/FlatBlack</material>
+    <material>Gazebo/DarkGrey</material>
+  </gazebo>
+  <gazebo reference="body_side_right">
+    <material>Gazebo/LightYellow</material>
+    <commandTopic>/turtle1/cmd_vel</commandTopic>
+  </gazebo>
+  <gazebo reference="body_side_left">
+    <material>Gazebo/LightYellow</material>
+    <commandTopic>/turtle1/cmd_vel</commandTopic>
   </gazebo>
   <gazebo reference="caster_back_right_link">
@@ -86,7 +94,7 @@
       <rightJoint>wheel_right_joint</rightJoint>
       <wheelSeparation>0.287</wheelSeparation>
-      <wheelDiameter>0.066</wheelDiameter>
+      <wheelDiameter>0.2</wheelDiameter>
       <wheelAcceleration>1</wheelAcceleration>
-      <wheelTorque>10</wheelTorque>
+      <wheelTorque>100</wheelTorque>
       <rosDebugLevel>na</rosDebugLevel>
     </plugin>

File: src/covid_robot_description/urdf/covid_robot.urdf.xacro (robot description, xacro)
@@ -10,9 +10,9 @@
     <parent link="base_footprint"/>
     <child link="base_link" />
-    <origin xyz="0 0 0.01" rpy="0 0 0"/>
+    <origin xyz="0 0 0.010" rpy="0 0 -1.57"/>
   </joint>
   <link name="base_link">
     <visual>
-      <origin xyz="0 0 0.25" rpy="0 0 0"/>
+      <origin xyz="0.0 0 0.25" rpy="0 0 0.0"/>
       <geometry>
         <mesh filename="package://covid_robot_description/meshes/bases/covid_robot_body.stl" scale="0.001 0.001 0.001"/>
@@ -21,24 +21,64 @@
     </visual>
     <collision>
-      <origin xyz="0.0 0 0.047" rpy="0 0 0"/>
-      <geometry>
-        <box size="1.0 1.0 0.093"/>
-      </geometry>
-    </collision>
-    <inertial>
-      <origin xyz="0 0 0" rpy="0 0 0"/>
-      <mass value="1.3729096e+00"/>
-      <inertia ixx="8.7002718e-03" ixy="-4.7576583e-05" ixz="1.1160499e-04"
-               iyy="8.6195418e-03" iyz="-3.5422299e-06"
-               izz="1.4612727e-02" />
+      <origin xyz="0 0 0.047" rpy="0 0 0"/>
+      <geometry>
+        <box size="0.266 0.266 0.094"/>
+      </geometry>
+    </collision>
+  </link>
+  <joint name="wheel_right_joint_1_steer" type="fixed">
+    <parent link="base_link"/>
+    <child link="wheel_right_link_1_steer"/>
+    <!-- if error => z = -0.03 -->
+    <origin xyz="-0.4 0.22 -0.08" rpy="0 0 0"/>
+  </joint>
+  <link name="wheel_right_link_1_steer">
+    <visual>
+      <origin xyz="0 0 0.1" rpy="1.57 0 0"/>
+      <geometry>
+        <mesh filename="package://covid_robot_description/meshes/wheels/steering_motor.stl" scale="0.001 0.001 0.001"/>
+      </geometry>
+      <material name="dark"/>
+    </visual>
+    <collision>
+      <origin xyz="0 0 0" rpy="0 0 0"/>
+    </collision>
+  </link>
+  <joint name="wheel_right_joint_1" type="continuous">
+    <parent link="base_link"/>
+    <child link="wheel_right_link_1"/>
+    <!-- x = -0.45 -->
+    <origin xyz="-0.48 0.22 0.023" rpy="0 -1.57 0"/>
+    <axis xyz="0 0 1"/>
+  </joint>
+  <link name="wheel_right_link_1">
+    <visual>
+      <origin xyz="0.0 0 0.02" rpy="1.57 0 0"/>
+      <geometry>
+        <mesh filename="package://covid_robot_description/meshes/wheels/covid_robot_tire.stl" scale="0.001 0.001 0.001"/>
+      </geometry>
+      <material name="dark"/>
+    </visual>
+    <collision>
+      <origin xyz="0 0 0" rpy="0 0 0"/>
+      <geometry>
+        <cylinder length="0.018" radius="0.1"/>
+      </geometry>
+    </collision>
+    <inertial>
+      <origin xyz="0 0 0" />
+      <mass value="2.8498940e-02" />
+      <inertia ixx="1.1175580e-05" ixy="-4.2369783e-11" ixz="-5.9381719e-09"
+               iyy="1.1192413e-05" iyz="-1.4400107e-11"
+               izz="2.0712558e-05" />
     </inertial>
   </link>
-  <joint name="wheel_left_joint_4_steer" type="fixed">
-    <parent link="base_link"/>
-    <child link="wheel_left_link_4_steer"/>
-    <origin xyz="-0.40 0.22 -0.03" rpy="0 0 0"/>
-  </joint>
-  <link name="wheel_left_link_4_steer">
-    <visual>
+  <joint name="wheel_left_joint_1_steer" type="fixed">
+    <parent link="base_link"/>
+    <child link="wheel_left_link_1_steer"/>
+    <origin xyz="0.40 0.22 -0.08" rpy="0 0 0"/>
+  </joint>
+  <link name="wheel_left_link_1_steer">
+      <visual>
       <origin xyz="0 0 0.1" rpy="1.57 0 0"/>
       <geometry>
@@ -51,11 +91,11 @@
     </collision>
   </link>
-  <joint name="wheel_left_joint_4" type="continuous">
-    <parent link="base_link"/>
-    <child link="wheel_left_link_4"/>
-    <origin xyz="-0.45 0.22 0.023" rpy="0 1.57 0"/>
+  <joint name="wheel_left_joint_1" type="continuous">
+    <parent link="base_link"/>
+    <child link="wheel_left_link_1"/>
+    <origin xyz="0.48 0.22 0.023" rpy="0 -1.57 0"/>
     <axis xyz="0 0 1"/>
   </joint>
-  <link name="wheel_left_link_4">
+  <link name="wheel_left_link_1">
     <visual>
       <origin xyz="0 0 0.02" rpy="1.57 0 0"/>
@@ -68,5 +108,5 @@
       <origin xyz="0 0 0" rpy="0 0 0"/>
       <geometry>
-        <cylinder length="0.018" radius="0.033"/>
+        <cylinder length="0.018" radius="0.1"/>
       </geometry>
     </collision>
@@ -82,8 +122,8 @@
     <parent link="base_link"/>
     <child link="wheel_left_link_steer"/>
-    <origin xyz="0.40 0.22 -0.03" rpy="0 0 0"/>
+    <origin xyz="0.40 -0.22 -0.08" rpy="0 0 0"/>
   </joint>
   <link name="wheel_left_link_steer">
-      <visual>
+    <visual>
       <origin xyz="0 0 0.1" rpy="1.57 0 0"/>
       <geometry>
@@ -99,10 +139,10 @@
     <parent link="base_link"/>
     <child link="wheel_left_link"/>
-    <origin xyz="0.45 0.22 0.023" rpy="0 -1.57 0"/>
+    <origin xyz="0.48 -0.22 0.023" rpy="0 -1.57 0"/>
     <axis xyz="0 0 1"/>
   </joint>
   <link name="wheel_left_link">
     <visual>
-      <origin xyz="0 0 0.02" rpy="1.57 0 0"/>
+      <origin xyz="0.0 0 0.02" rpy="1.57 0 0"/>
       <geometry>
         <mesh filename="package://covid_robot_description/meshes/wheels/covid_robot_tire.stl" scale="0.001 0.001 0.001"/>
@@ -113,5 +153,5 @@
       <origin xyz="0 0 0" rpy="0 0 0"/>
       <geometry>
-        <cylinder length="0.018" radius="0.033"/>
+        <cylinder length="0.018" radius="0.1"/>
       </geometry>
     </collision>
@@ -127,5 +167,5 @@
     <parent link="base_link"/>
     <child link="wheel_right_link_steer"/>
-    <origin xyz="0.40 -0.22 -0.03" rpy="0 0 0"/>
+    <origin xyz="-0.40 -0.22 -0.08" rpy="0 0 0"/>
   </joint>
   <link name="wheel_right_link_steer">
@@ -144,5 +184,5 @@
     <parent link="base_link"/>
     <child link="wheel_right_link"/>
-    <origin xyz="0.45 -0.22 0.023" rpy="0 -1.57 0"/>
+    <origin xyz="-0.48 -0.22 0.023" rpy="0 -1.57 0"/>
     <axis xyz="0 0 1"/>
   </joint>
@@ -153,10 +193,9 @@
         <mesh filename="package://covid_robot_description/meshes/wheels/covid_robot_tire.stl" scale="0.001 0.001 0.001"/>
       </geometry>
-      <material name="dark"/>
-    </visual>
-    <collision>
-      <origin xyz="0 0 0" rpy="0 0 0"/>
-      <geometry>
-        <cylinder length="0.018" radius="0.033"/>
+    </visual>
+    <collision>
+      <origin xyz="0 0 0" rpy="0 0 0"/>
+      <geometry>
+        <cylinder length="0.018" radius="0.1"/>
       </geometry>
     </collision>
@@ -169,56 +208,50 @@
       </inertial>
   </link>
-  <joint name="wheel_right_joint_1_steer" type="fixed">
-    <parent link="base_link"/>
-    <child link="wheel_right_link_1_steer"/>
-    <origin xyz="-0.40 -0.22 -0.03" rpy="0 0 0"/>
-  </joint>
-  <link name="wheel_right_link_1_steer">
-    <visual>
-      <origin xyz="0 0 0.1" rpy="1.57 0 0"/>
-      <geometry>
-        <mesh filename="package://covid_robot_description/meshes/wheels/steering_motor.stl" scale="0.001 0.001 0.001"/>
-      </geometry>
-      <material name="dark"/>
-    </visual>
-    <collision>
-      <origin xyz="0 0 0" rpy="0 0 0"/>
-    </collision>
-  </link>
-  <joint name="wheel_right_joint_1" type="continuous">
-    <parent link="base_link"/>
-    <child link="wheel_right_link_1"/>
-    <origin xyz="-0.45 -0.22 0.023" rpy="0 1.57 0"/>
-    <axis xyz="0 0 1"/>
-  </joint>
-  <link name="wheel_right_link_1">
-    <visual>
-      <origin xyz="0 0 0.02" rpy="1.57 0 0"/>
-      <geometry>
-        <mesh filename="package://covid_robot_description/meshes/wheels/covid_robot_tire.stl" scale="0.001 0.001 0.001"/>
-      </geometry>
-    </visual>
-    <collision>
-      <origin xyz="0 0 0" rpy="0 0 0"/>
-      <geometry>
-        <cylinder length="0.018" radius="0.033"/>
-      </geometry>
-    </collision>
-    <inertial>
-      <origin xyz="0 0 0" />
-      <mass value="2.8498940e-02" />
-      <inertia ixx="1.1175580e-05" ixy="-4.2369783e-11" ixz="-5.9381719e-09"
-               iyy="1.1192413e-05" iyz="-1.4400107e-11"
-               izz="2.0712558e-05" />
-      </inertial>
+  <joint name="body_side_left_rack" type="fixed">
+    <parent link="base_link"/>
+    <child link="body_side_left_rack"/>
+    <!-- x = -0.45 when opened -->
+    <origin xyz="-0.45 0.0 0.9" rpy="0 0 0"/>
+  </joint>
+  <link name="body_side_left_rack">
+    <visual>
+      <origin xyz="0.0 0.0 0.0" rpy="0 -1.65 0"/>
+      <geometry>
+        <mesh filename="package://covid_robot_description/meshes/bases/body_side_rack.stl" scale="0.001 0.001 0.001"/>
+      </geometry>
+      <material name="dark"/>
+    </visual>
+    <collision>
+      <origin xyz="0 0 0" rpy="0 0 0"/>
+    </collision>
+  </link>
+  <joint name="body_side_right_rack" type="fixed">
+    <parent link="base_link"/>
+    <child link="body_side_right_rack"/>
+    <!-- x = 0.45 when opened -->
+    <origin xyz="0.45 0.0 0.9" rpy="0 0 0"/>
+  </joint>
+  <link name="body_side_right_rack">
+    <visual>
+      <origin xyz="0.0 0.0 0.0" rpy="0 -1.65 0"/>
+      <geometry>
+        <mesh filename="package://covid_robot_description/meshes/bases/body_side_rack.stl" scale="0.001 0.001 0.001"/>
+      </geometry>
+      <material name="dark"/>
+    </visual>
+    <collision>
+      <origin xyz="0 0 0" rpy="0 0 0"/>
+    </collision>
   </link>
   <joint name="body_side_left" type="fixed">
     <parent link="base_link"/>
     <child link="body_side_left"/>
-    <origin xyz="-0.30 0.0 0.460" rpy="0 0 0"/>
+    <!-- x = -0.45 when closed -->
+    <!-- x = -0.75 when opened -->
+    <origin xyz="-0.45 0.0 0.460" rpy="0 0 0"/>
   </joint>
   <link name="body_side_left">
     <visual>
-      <origin xyz="-0.3 0.1 0.1" rpy="1.57 0 0"/>
+      <origin xyz="0.0 0.0 0.1" rpy="1.57 0 0"/>
       <geometry>
         <mesh filename="package://covid_robot_description/meshes/bases/body_side.stl" scale="0.001 0.001 0.001"/>
@@ -233,9 +266,11 @@
     <parent link="base_link"/>
     <child link="body_side_right"/>
-    <origin xyz="0.30 0.0 0.460" rpy="0 0 0"/>
+    <!-- x = 0.45 when closed -->
+    <!-- x = 0.75 when opened -->
+    <origin xyz="0.45 0.0 0.460" rpy="0 0 0"/>
   </joint>
   <link name="body_side_right">
     <visual>
-      <origin xyz="0.1 0.1 0.1" rpy="1.57 0 0"/>
+      <origin xyz="0.0 0.0 0.1" rpy="1.57 0 -3.14"/>
       <geometry>
         <mesh filename="package://covid_robot_description/meshes/bases/body_side.stl" scale="0.001 0.001 0.001"/>
@@ -246,36 +281,66 @@
     </collision>
   </link>
-  <joint name="body_side_rack_left" type="fixed">
-    <parent link="base_link"/>
-    <child link="body_side_rack_left"/>
-    <origin xyz="-0.30 0.0 0.835" rpy="0 1.57 1.57"/>
-  </joint>
-  <link name="body_side_rack_left">
-    <visual>
-      <origin xyz="0 0 0.1" rpy="1.57 0 0"/>
-      <geometry>
-        <mesh filename="package://covid_robot_description/meshes/bases/body_side_rack.stl" scale="0.001 0.001 0.001"/>
-      </geometry>
-      <material name="dark"/>
-    </visual>
-    <collision>
-      <origin xyz="0 0 0" rpy="0 0 0"/>
-    </collision>
-  </link>
-  <joint name="caster_back_right_joint" type="fixed">
-    <parent link="base_link"/>
-    <child link="caster_back_right_link"/>
-    <origin xyz="-0.177 -0.064 -0.004" rpy="-1.57 0 0"/>
-  </joint>
-  <link name="caster_back_right_link">
-    <collision>
-      <origin xyz="0 0.001 0" rpy="0 0 0"/>
-      <geometry>
-        <box size="0.030 0.009 0.020"/>
-      </geometry>
-    </collision>
-    <inertial>
-      <origin xyz="0 0 0" />
-      <mass value="0.005" />
+  <!-- <joint name="left_cleaning" type="fixed">
+    <parent link="base_link"/>
+    <child link="left_cleaning"/>
+    <origin xyz="-0.9 0.1 .5" rpy="0 0 0"/>
+  </joint>
+  <link name="left_cleaning">
+    <visual>
+      <origin xyz="0.0 0.0 0.0" rpy="1.57 0 0"/>
+      <geometry>
+        <mesh filename="package://covid_robot_description/meshes/bases/cleaning.stl" scale="0.001 0.001 0.001"/>
+      </geometry>
+      <material name="dark"/>
+    </visual>
+    <collision>
+      <origin xyz="0 0 0" rpy="0 0 0"/>
+    </collision>
+  </link>
+  <joint name="right_cleaning" type="fixed">
+    <parent link="base_link"/>
+    <child link="right_cleaning"/>
+    <origin xyz="0.65 0.1 0.5" rpy="1.57 0 0"/>
+  </joint>
+  <link name="right_cleaning">
+    <visual>
+      <origin xyz="0.0 0.0 0.0" rpy="0 0 0"/>
+      <geometry>
+        <mesh filename="package://covid_robot_description/meshes/bases/cleaning.stl" scale="0.001 0.001 0.001"/>
+      </geometry>
+      <material name="dark"/>
+    </visual>
+    <collision>
+      <origin xyz="0 0 0" rpy="0 0 0"/>
+    </collision>
+  </link> -->
+  <joint name="imu_joint" type="fixed">
+    <parent link="base_link"/>
+    <child link="imu_link"/>
+    <origin xyz="0.0 0 0.068" rpy="0 0 0"/>
+  </joint>
+  <link name="imu_link"/>
+  <joint name="scan_joint" type="fixed">
+    <parent link="base_link"/>
+    <child link="base_scan"/>
+    <origin xyz="0.0 0 0.2" rpy="0 0 1.57"/>
+  </joint>
+  <link name="base_scan">
+    <visual>
+      <origin xyz="0 0 0" rpy="0 0 0"/>
+      <geometry>
+        <mesh filename="package://turtlebot3_description/meshes/sensors/lds.stl" scale="0.001 0.001 0.001"/>
+      </geometry>
+      <material name="dark"/>
+    </visual>
+    <collision>
+      <origin xyz="0.015 0 -0.0065" rpy="0 0 0"/>
+      <geometry>
+        <cylinder length="0.0315" radius="0.055"/>
+      </geometry>
+    </collision>
+    <inertial>
+      <mass value="0.114" />
+      <origin xyz="0 0 0" />
       <inertia ixx="0.001" ixy="0.0" ixz="0.0"
                iyy="0.001" iyz="0.0"
@@ -283,56 +348,29 @@
     </inertial>
   </link>
-  <joint name="caster_back_left_joint" type="fixed">
-    <parent link="base_link"/>
-    <child link="caster_back_left_link"/>
-    <origin xyz="-0.177 0.064 -0.004" rpy="-1.57 0 0"/>
-  </joint>
-  <link name="caster_back_left_link">
-    <collision>
-      <origin xyz="0 0.001 0" rpy="0 0 0"/>
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
File: src/covid_robot_description/urdf/turtlebot3_waffle.urdf.xacro (robot description, xacro)
@@ -2,5 +2,5 @@
 <robot name="turtlebot3_waffle" xmlns:xacro="http://ros.org/wiki/xacro">
   <xacro:include filename="$(find turtlebot3_description)/urdf/common_properties.xacro"/>
-  <xacro:include filename="$(find turtlebot3_description)/urdf/turtlebot3_waffle.gazebo.xacro"/>
+  <xacro:include filename="$(find covid_robot_description)/urdf/covid_robot.gazebo.xacro"/>
   <xacro:property name="r200_cam_rgb_px" value="0.005"/>
   <xacro:property name="r200_cam_rgb_py" value="0.018"/>
@@ -19,5 +19,5 @@
         <mesh filename="package://turtlebot3_description/meshes/bases/waffle_base.stl" scale="0.001 0.001 0.001"/>
       </geometry>
-      <material name="light_black"/>
+      <material>Gazebo/BlueTransparent</material>
     </visual>
     <collision>
@@ -46,5 +46,5 @@
         <mesh filename="package://covid_robot_description/meshes/bases/total_assemble.stl" scale="0.001 0.001 0.001"/>
       </geometry>
-      <material name="dark"/>
+      <material name="black"/>
     </visual>
     <collision>
@@ -64,5 +64,5 @@
         <mesh filename="package://turtlebot3_description/meshes/wheels/left_tire.stl" scale="0.001 0.001 0.001"/>
       </geometry>
-      <material name="dark"/>
+      <material name="black"/>
     </visual>
     <collision>
@@ -92,5 +92,5 @@
         <mesh filename="package://turtlebot3_description/meshes/wheels/right_tire.stl" scale="0.001 0.001 0.001"/>
       </geometry>
-      <material name="dark"/>
+      <material name="black"/>
     </visual>
     <collision>
